File: usb_hub.kicad_sch (KiCad schematic)
At the start: 11 parts, among them J1 USB_C_Receptacle_USB2.0_16P, J2 Barrel_Jack_Switch, U1 USB2514B_Bi, U2 SPX3819M5-L

Commit message: Modified schematic
Parts:
- added C10, C11, C12, C7, C8, C9: 100nF, symbol Device:C
- added C5, C6: 2.2uF, symbol Device:C
- added FB2: 120R/3A, symbol Device:FerriteBead
- added R2, R3: 5.1K, symbol Device:R
- added U3: USBLC6-2SC6, Package_TO_SOT_SMD:SOT-23-6, symbol Power_Protection:USBLC6-2SC6
- FB1: value 3A -> 120R/3A
- R1: value 330 -> 330R
Connections:
- net GND: now also J1.A1 (GND), J1.A12 (GND), J1.B1 (GND), J1.B12 (GND), J1.SH (SHIELD), U1.10 (VDDA33), U1.15 (VDD33), U1.23 (VDD33), U1.29 (VDDA33), U1.36 (VDDA33), U1.5 (VDDA33), C10.2, C11.2, C12.2, C5.2, C6.2, C7.2, C8.2, C9.2, R2.2, R3.2, U3.2 (GND); no longer U2.3 (EN)
- net +5V FILT: now reaches C4.1, FB1.2, U2.1 (IN)
- net +5V FILT: now also C6.1, FB2.2
- net +3.3V: now reaches D1.1 (K), R1.1
- net +3.3V: now also C10.1, C11.1, C12.1, C7.1, C8.1, C9.1
- net +5V HOST: now reaches J1.A4 (VBUS), J1.A9 (VBUS), J1.B4 (VBUS), J1.B9 (VBUS)
- net +5V HOST: now also C5.1, FB2.1, U3.5 (VBUS)
- net at J1.A5 (CC1): now also R2.1
- net USB CONN HOST D+: now reaches J1.A6 (D+)
- net USB CONN HOST D+: now also J1.B6 (D+), U1.31 (USBDP_UP), U3.6 (I/O1)
- net USB CONN HOST D-: now reaches J1.A7 (D-)
- net USB CONN HOST D-: now also J1.B7 (D-), U1.30 (USBDM_UP), U3.4 (I/O2)
- net at J1.B5 (CC2): now also R3.1
- net VBUS_DET: now reaches U1.27 (VBUS_DET)
- net VBUS_DET: now also U2.3 (EN)
- no-connect marks 0 -> 2
Other:
- note added: "USB Hub Section"
- note removed: "Microcontroller Section"
- moved on the sheet: J1

Commit message: Made connections to pins of USB Hub
Parts:
- added C13: 0.1uF, symbol Device:C
- added R4: 12k, symbol Device:R
- added R5, R6: 100k, symbol Device:R
Connections:
- net +3.3V: now also R5.2
- net GND: now also U1.37 (VSS), C13.1, R4.1, R6.1
- net USB CONN HOST D+: now also U3.1 (I/O1)
- net USB CONN HOST D-: now also U3.3 (I/O2)
- net VBUS_DET: now also R5.1, R6.2
- net at U1.14 (CRFILT): now also U1.34 (PLLFILT), C13.2
- net at U1.35 (RBIAS): now also R4.2
Other:
- moved on the sheet: U3

Commit message: Added modification to schematic
Parts:
- removed C5, C6: 2.2uF, symbol Device:C
- removed FB2: 120R/3A, symbol Device:FerriteBead
- added C14, C15: 10pF, symbol Device:C
- added D2: LED, symbol Device:LED
- added R7: 47k, symbol Device:R
- added Y1: 24MHz, symbol Device:Crystal
Connections:
- net +3.3V: now also D2.2 (A), R7.2
- net GND: now also C14.1, C15.1
- net at U1.25 (HS_IND/CFG_SEL1): now also D2.1 (K), R7.1
- net at U1.32 (XTALOUT): now also C14.2, Y1.1
- net at U1.33 (XTALIN/CLKIN): now also C15.2, Y1.2
Other:
- moved on the sheet: C13, J1, R2, R3, R4, R5, R6, U3

Commit message: Updated Schematic
Parts:
- removed FB1: 120R/3A, symbol Device:FerriteBead
- added L1: L, symbol Device:L
Connections:
- net +3.3V: now also C1.1, D1.2 (A), U2.5 (OUT); no longer D1.1 (K), R1.1
- net +5V: now also L1.1
- net +5V FILT: now also L1.2
- net USB CONN HOST D+: now also U1.2 (USBDP_DN1/PRT_DIS_P1), U1.4 (USBDP_DN2/PRT_DIS_P2), U1.7 (USBDP_DN3/PRT_DIS_P3), U1.9 (USBDP_DN4/PRT_DIS_P4)
- net USB CONN HOST D-: now also U1.1 (USBDM_DN1/PRT_DIS_M1), U1.3 (USBDM_DN2/PRT_DIS_M2), U1.6 (USBDM_DN3/PRT_DIS_M3), U1.8 (USBDM_DN4/PRT_DIS_M4)
- new net: D1.1 (K), R1.1
Changed lines of the file:
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@@
 	(text "USB Hub Section"
 		(exclude_from_sim no)
-		(at 289.814 14.986 0)
+		(at 255.27 14.732 0)
 		(effects
 			(font
@@
 	)
 	(junction
-		(at 134.62 35.56)
-		(diameter 0)
-		(color 0 0 0 0)
-	)
-	(junction
 		(at 257.81 71.12)
 		(diameter 0)
@@
 	)
 	(junction
+		(at 113.03 35.56)
+		(diameter 0)
+		(color 0 0 0 0)
+	)
+	(junction
 		(at 107.95 35.56)
 		(diameter 0)
@@
 	(wire
 		(pts
-			(xy 134.62 34.29) (xy 134.62 35.56)
+			(xy 318.77 30.48) (xy 328.93 30.48)
 		)
 		(stroke
@@
 	(wire
 		(pts
-			(xy 318.77 30.48) (xy 328.93 30.48)
+			(xy 273.05 78.74) (xy 285.75 78.74)
 		)
 		(stroke
@@
 	(wire
 		(pts
-			(xy 273.05 78.74) (xy 285.75 78.74)
+			(xy 113.03 31.75) (xy 113.03 35.56)
 		)
 		(stroke
@@
 	(wire
 		(pts
-			(xy 107.95 35.56) (xy 118.11 35.56)
+			(xy 107.95 35.56) (xy 113.03 35.56)
 		)
 		(stroke
@@
 	(wire
 		(pts
+			(xy 113.03 35.56) (xy 118.11 35.56)
+		)
+		(stroke
+			(width 0)
+			(type default)
+		)
+	)
+	(wire
+		(pts
 			(xy 50.8 99.06) (xy 50.8 100.33)
 		)
@@
 	)
 	(label "USB CONN HOST D-"
+		(at 367.03 48.26 0)
+		(effects
+			(font
+				(size 1.27 1.27)
+			)
+			(justify left bottom)
+		)
+	)
+	(label "USB CONN HOST D+"
+		(at 367.03 50.8 0)
+		(effects
+			(font
+				(size 1.27 1.27)
+			)
+			(justify left bottom)
+		)
+	)
+	(label "USB CONN HOST D-"
+		(at 367.03 73.66 0)
+		(effects
+			(font
+				(size 1.27 1.27)
+			)
+			(justify left bottom)
+		)
+	)
+	(label "USB CONN HOST D-"
 		(at 109.22 92.71 0)
 		(effects
@@
 		)
 	)
+	(label "USB CONN HOST D-"
+		(at 367.03 86.36 0)
+		(effects
+			(font
+				(size 1.27 1.27)
+			)
+			(justify left bottom)
+		)
+	)
+	(label "USB CONN HOST D+"
+		(at 367.03 88.9 0)
+		(effects
+			(font
+				(size 1.27 1.27)
+			)
+			(justify left bottom)
+		)
+	)
 	(label "USB CONN HOST D+"
 		(at 80.01 90.17 0)
@@
 	)
 	(label "USB CONN HOST D+"
+		(at 367.03 63.5 0)
+		(effects
+			(font
+				(size 1.27 1.27)
+			)
+			(justify left bottom)
+		)
+	)
+	(label "USB CONN HOST D+"
 		(at 290.83 55.88 0)
 		(effects
@@
 		)
 	)
+	(label "USB CONN HOST D-"
+		(at 367.03 60.96 0)
+		(effects
+			(font
+				(size 1.27 1.27)
+			)
+			(justify left bottom)
+		)
+	)
 	(label "VBUS_DET"
 		(at 64.77 59.69 0)
@@
 		)
 	)
+	(label "USB CONN HOST D+"
+		(at 367.03 76.2 0)
+		(effects
+			(font
+				(size 1.27 1.27)
+			)
+			(justify left bottom)
+		)
+	)
 	(symbol
 		(lib_id "power:GND")
@@
 	(symbol
 		(lib_id "power:+3.3V")
-		(at 134.62 34.29 0)
+		(at 113.03 31.75 0)
 		(unit 1)
 		(body_style 1)
@@
 		(fields_autoplaced yes)
 		(property "Reference" "#PWR04"
-			(at 134.62 38.1 0)
+			(at 113.03 35.56 0)
 			(hide yes)
 			(show_name no)
@@
 		)
 		(property "Value" "+3.3V"
-			(at 134.62 29.21 0)
+			(at 113.03 26.67 0)
 			(show_name no)
 			(do_not_autoplace no)
@@
 		)
 		(property "Footprint" ""
-			(at 134.62 34.29 0)
+			(at 113.03 31.75 0)
 			(hide yes)
 			(show_name no)
@@
 		)
 		(property "Datasheet" ""
-			(at 134.62 34.29 0)
+			(at 113.03 31.75 0)
 			(hide yes)
 			(show_name no)
@@
 		)
 		(property "Description" "Power symbol creates a global label with name \"+3.3V\""
-			(at 134.62 34.29 0)
+			(at 113.03 31.75 0)
 			(hide yes)
 			(show_name no)
@@
 	)
 	(symbol
-		(lib_id "Device:FerriteBead")
-		(at 58.42 35.56 90)
-		(unit 1)
-		(body_style 1)
-		(exclude_from_sim no)
-		(in_bom yes)
-		(on_board yes)
-		(in_pos_files yes)
-		(dnp no)
-		(fields_autoplaced yes)
-		(property "Reference" "FB1"
-			(at 58.3692 27.94 90)
-			(show_name no)
-			(do_not_autoplace no)
-			(effects
-				(font
-					(size 1.27 1.27)
-				)
-			)
-		)
-		(property "Value" "120R/3A"
-			(at 58.3692 30.48 90)
-			(show_name no)
-			(do_not_autoplace no)
-			(effects
-				(font
-					(size 1.27 1.27)
-				)
-			)
-		)
-		(property "Footprint" ""
-			(at 58.42 37.338 90)
-			(hide yes)
-			(show_name no)
-			(do_not_autoplace no)
-			(effects
-				(font
-					(size 1.27 1.27)
-				)
-			)
-		)
-		(property "Datasheet" ""
-			(at 58.42 35.56 0)
-			(hide yes)
-			(show_name no)
-			(do_not_autoplace no)
-			(effects
-				(font
-					(size 1.27 1.27)
-				)
-			)
-		)
-		(property "Description" "Ferrite bead"
-			(at 58.42 35.56 0)
-			(hide yes)
-			(show_name no)
-			(do_not_autoplace no)
-			(effects
-				(font
-					(size 1.27 1.27)
-				)
-			)
-		)
-		(pin "2"
-		)
-		(pin "1"
-		)
-		(instances
-			(project "usb_hub"
-				(path "/f1456d5d-56e0-456f-ac13-d857f76447dd"
-					(reference "FB1")
-					(unit 1)
-				)
-			)
-		)
-	)
-	(symbol
 		(lib_id "Device:LED")
 		(at 121.92 35.56 180)
@@
 					(unit 1)
 				)
+			)
+		)
+	)
+	(symbol
+		(lib_id "Device:L")
+		(at 58.42 35.56 90)
+		(unit 1)
+		(body_style 1)
+		(exclude_from_sim no)
+		(in_bom yes)
+		(on_board yes)
+		(in_pos_files yes)
+		(dnp no)
+		(fields_autoplaced yes)
+		(property "Reference" "L1"
+			(at 58.42 30.48 90)
+			(show_name no)
+			(do_not_autoplace no)
+			(effects
+				(font
+					(size 1.27 1.27)
+				)
+			)
+		)
+		(property "Value" "L"
+			(at 58.42 33.02 90)
+			(show_name no)
+			(do_not_autoplace no)
+			(effects
+				(font
+					(size 1.27 1.27)
+				)
+			)
+		)
+		(property "Footprint" ""
+			(at 58.42 35.56 0)
+			(hide yes)
+			(show_name no)
+			(do_not_autoplace no)
+			(effects
+				(font
+					(size 1.27 1.27)
+				)
+			)
+		)
+		(property "Datasheet" ""
+			(at 58.42 35.56 0)
+			(hide yes)
+			(show_name no)
+			(do_not_autoplace no)
+			(effects
+				(font
+					(size 1.27 1.27)
+				)
+			)
+		)
+		(property "Description" "Inductor"
+			(at 58.42 35.56 0)
+			(hide yes)
+			(show_name no)
+			(do_not_autoplace no)
+			(effects
+				(font
+					(size 1.27 1.27)
+				)
+			)
+		)
+		(pin "1"
+		)
+		(pin "2"
+		)
+		(instances
+			(project "usb_hub"
+				(path "/f1456d5d-56e0-456f-ac13-d857f76447dd"
+					(reference "L1")
+					(unit 1)
+				)
